File: pcb/pico-folio-keyboard.kicad_pcb (KiCad board)
At the start: 2 copper layers, 205.1 x 68.4 mm, 133 parts, among them SW1 SW_Push, SW10 SW_Push, SW11 SW_Push, SW12 SW_Push, SW13 SW_Push, SW14 SW_Push, SW15 SW_Push, SW16 SW_Push, SW17 SW_Push, SW18 SW_Push, SW19 SW_Push, SW2 SW_Push, SW20 SW_Push, SW21 SW_Push, SW22 SW_Push, SW23 SW_Push, SW24 SW_Push, SW25 SW_Push, SW26 SW_Push, SW27 SW_Push, SW28 SW_Push, SW29 SW_Push, SW3 SW_Push, SW30 SW_Push, SW31 SW_Push, SW32 SW_Push, SW33 SW_Push, SW34 SW_Push, SW35 SW_Push, SW36 SW_Push, SW37 SW_Push, SW38 SW_Push, SW39 SW_Push, SW4 SW_Push, SW40 SW_Push, SW41 SW_Push, SW42 SW_Push, SW43 SW_Push, SW44 SW_Push, SW45 SW_Push, SW46 SW_Push, SW47 SW_Push, SW48 SW_Push, SW49 SW_Push, SW5 SW_Push, SW50 SW_Push, SW51 SW_Push, SW52 SW_Push, SW53 SW_Push, SW54 SW_Push, SW55 SW_Push, SW56 SW_Push, SW57 SW_Push, SW58 SW_Push, SW59 SW_Push, SW6 SW_Push, SW60 SW_Push, SW61 SW_Push, SW62 SW_Push, SW63 SW_Push, SW64 SW_Push, SW7 SW_Push, SW8 SW_Push, SW9 SW_Push

Commit message: updated schematic and pcb to break out vbus and gnd for usb without bodge wires
Parts:
- added J1: Conn_01x02_Pin, Connector_PinHeader_2.54mm:PinHeader_1x02_P2.54mm_Vertical, F.Cu at (58.0, 85.0)
Connections:
- A1 pad 13: unconnected-(A1-GND-Pad13)_1 -> Net-(J1-Pin_1)
- A1 pad 18: unconnected-(A1-GND-Pad13)_2 -> Net-(J1-Pin_1)
- A1 pad 23: unconnected-(A1-GND-Pad13)_4 -> Net-(J1-Pin_1)
- A1 pad 28: unconnected-(A1-GND-Pad13)_6 -> Net-(J1-Pin_1)
- A1 pad 3: unconnected-(A1-GND-Pad13) -> Net-(J1-Pin_1)
- A1 pad 38: unconnected-(A1-GND-Pad13)_5 -> Net-(J1-Pin_1)
- A1 pad 40: unconnected-(A1-VBUS-Pad40) -> Net-(A1-VBUS)
- A1 pad 8: unconnected-(A1-GND-Pad13)_3 -> Net-(J1-Pin_1)
Routing:
- net Net-(A1-VBUS): track 0.00 -> 14.4 mm
- net Net-(J1-Pin_1): track 0.00 -> 11.3 mm
